File: Mbc3-Flash-Storage-PCB.kicad_pcb (KiCad board)
At the start: 2 copper layers, 51 x 60.7 mm, 27 parts, among them U0 CartBus, U2 MBC3, U3 FM18W08, U4 BA6129AF, U5 74LVC1G332GW,125, Y1 Crystal

Commit message: Replaced 3 input or-gate with a 2-input one.
Parts:
- removed REF**: OSHW-Logo_5.7x6mm_Copper, Symbol:OSHW-Logo_5.7x6mm_Copper
- R1: value 300Kohm -> 330Kohm
- U5: value 74LVC1G332GW,125 -> 74LVC1G32
Connections:
- U5 pad 2: GND -> CLK
- U5 pad 3: CLK -> GND
- U5 pad 6: CS -> VCC
Routing:
- net CS: track 22.7 -> 0.00 mm
- net GND: track 188.6 -> 197.3 mm, vias 15 -> 17
- net VCC: track 135.4 -> 135.9 mm
Other:
- board text added: "DMG-KGDU-10+"
- board text added: "HDR"
- board text added: "M.H 22"
- board text removed: "2022 W.P"
- board text removed: "MBC-FLSH-3"
