File: KiCad Files/DMG-KGDU-10+.kicad_pcb (KiCad board)
At the start: 2 copper layers, 51 x 60.7 mm, 26 parts, among them U0 CartBus, U2 MBC3, U3 FM18W08, U4 BA6129AF, U5 74LVC1G32, Y1 Crystal

Commit message: Rev 1.1 update
Parts:
- removed the R3 at (161.1, 95.3)
- moved R3 6.13 mm to (137.0, 85.6), turned to 180 degrees
- moved R2 1.65 mm to (140.8, 100.7), turned to 90 degrees
- moved C7 1.41 mm to (122.9, 108.2)
- moved C2 0.84 mm to (161.9, 116.5)
Routing:
- net GND: track 197.3 -> 189.5 mm
- net Net-(SW1-Pad2): track 6.09 -> 0.00 mm, vias 2 -> 0
- net VCC: track 135.9 -> 141.1 mm
- net RA14: track 44.2 -> 39.2 mm
- net BT+: track 78.3 -> 83.2 mm
- net RA17: track 51.3 -> 47.4 mm
- net RESET: track 59.1 -> 61.3 mm
- net A13: track 72.6 -> 70.8 mm
- net Vbatt: track 37.2 -> 38.9 mm
- net D3: track 74.1 -> 72.5 mm
- net \RST: track 26.0 -> 24.6 mm
- net A11: track 52.9 -> 53.7 mm
- net #CE: track 28.5 -> 29.3 mm
- net D0: track 69.3 -> 68.7 mm
- net D2: track 75.2 -> 74.7 mm
Other:
- board text added: "2-in OR"
- board text added: "BA6129AF"
- board text added: "FM18W08"
- board text added: "GND"
- board text added: "Rev 1.1"
- board text added: "TSOP II 44 MASK ROM"
- board text added: "VCC"
- board text removed: "1 5"
- board text removed: "R4 (Jumper)"
